File: motorcin.kicad_pcb (KiCad board)
At the start: 2 copper layers, 18 parts, among them J1 AC 24V, J3 Conn_01x04, SW1 SW_Push, U1 ATmega328P-P, Y1 16MHz

Commit message: arreglos esteticos etc
Parts:
- removed J3: Conn_01x04, Connector_PinSocket_2.54mm:PinSocket_1x04_P2.54mm_Vertical
- added C3: 22pF, Capacitor_THT:C_Disc_D5.0mm_W2.5mm_P5.00mm, F.Cu at (112.5, 128.5)
- added J2: Motor, Connector_PinSocket_2.54mm:PinSocket_1x04_P2.54mm_Vertical, F.Cu at (146.4, 141.0)
- C1: value 22pF -> 470μF; footprint Capacitor_THT:C_Radial_D5.0mm_H5.0mm_P2.00mm -> Capacitor_THT:CP_Radial_D8.0mm_P2.50mm
- C2: footprint Capacitor_THT:C_Radial_D5.0mm_H5.0mm_P2.00mm -> Capacitor_THT:C_Disc_D5.0mm_W2.5mm_P5.00mm
- J1: footprint TestPoint:TestPoint_2Pads_Pitch2.54mm_Drill0.8mm -> Connector_PinHeader_2.00mm:PinHeader_1x02_P2.00mm_Horizontal
- SW1: footprint Button_Switch_SMD:SW_Push_1TS009xxxx-xxxx-xxxx_6x6x5mm -> Button_Switch_SMD:SW_SPST_CK_RS282G05A3
- moved J1 105.7 mm to (184.5, 143.0), turned to 180 degrees
- moved D4 83.6 mm to (187.0, 135.0)
- moved D2 83.5 mm to (171.8, 135.0)
- moved D3 80.7 mm to (186.9, 125.0)
- moved D1 80.5 mm to (171.9, 125.0)
- moved SW1 73.6 mm to (109.5, 112.0)
- moved H2 58.9 mm to (152.9, 115.9)
- moved C1 58.6 mm to (163.7, 143.0), turned to 180 degrees
- moved R2 55.5 mm to (134.8, 129.5)
- moved H1 53.4 mm to (152.9, 99.4)
- moved Y1 48.5 mm to (117.5, 123.6)
- moved U1 48.0 mm to (123.2, 104.3)
- moved R1 45.2 mm to (116.5, 104.0)
- moved C2 42.8 mm to (112.5, 123.5), turned to 180 degrees
- moved A1 25.3 mm to (141.4, 135.5), turned to 90 degrees
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Connections:
- net Net-(U1-~{RESET}/PC6) renamed /RESET
- A1 pad 3: Net-(A1-A2) -> /MotA2
- A1 pad 4: Net-(A1-A1) -> /MotA1
- A1 pad 5: Net-(A1-B1) -> /MotB1
- A1 pad 6: Net-(A1-B2) -> /MotB2
- C1 pad 1: /CRISTAL 1 -> VCC_MOT
- C1 pad 2: GND -> GND_MOT
- C2 pad 1: /CRISTAL 2 -> /CRISTAL 1
- D2 pad 1: VCC_MOT -> unconnected-(D2-K-Pad1)
- D4 pad 2: GND_MOT -> unconnected-(D4-A-Pad2)
Routing:
- net VCC: track 0.00 -> 132.5 mm, vias 0 -> 2
- net GND: track 0.00 -> 82.0 mm, vias 0 -> 3
- net /BOTON: track 0.00 -> 81.3 mm, vias 0 -> 1
- net GND_MOT: track 18.7 -> 86.0 mm, vias 0 -> 2
- net /ENABLE: track 0.00 -> 33.0 mm, vias 0 -> 2
- net /STEP: track 0.00 -> 26.5 mm
- net /DIR: track 0.00 -> 21.2 mm
- net ACn_MOT: track 27.6 -> 14.4 mm
- net VCC_MOT: track 59.6 -> 69.7 mm, vias 2 -> 0
- net AC_MOT: track 25.4 -> 32.8 mm
- net /CRISTAL 1: track 5.95 -> 11.6 mm
- net /MotB2: track 0.00 -> 5.53 mm
- net /MotA2: track 0.00 -> 5.53 mm
- net /MotA1: track 0.00 -> 5.53 mm
- net /MotB1: track 0.00 -> 5.53 mm
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