File: motorcin.kicad_sch (KiCad schematic)
At the start: 18 parts, among them J1 AC 24V, J3 Conn_01x04, SW1 SW_Push, U1 ATmega328P-P, Y1 16MHz

Commit message: arreglos esteticos etc
Parts:
- removed C1: 22pF, Capacitor_THT:C_Radial_D5.0mm_H5.0mm_P2.00mm, symbol Device:C
- added C1: 470μF, Capacitor_THT:CP_Radial_D8.0mm_P2.50mm, symbol Device:C_Polarized
- added C3: 22pF, Capacitor_THT:C_Disc_D5.0mm_W2.5mm_P5.00mm, symbol Device:C
- added M1: Nema17, symbol Motor:Stepper_Motor_bipolar
- C2: footprint Capacitor_THT:C_Radial_D5.0mm_H5.0mm_P2.00mm -> Capacitor_THT:C_Disc_D5.0mm_W2.5mm_P5.00mm
- J1: footprint TestPoint:TestPoint_2Pads_Pitch2.54mm_Drill0.8mm -> Connector_PinHeader_2.00mm:PinHeader_1x02_P2.00mm_Horizontal
- J2: renamed from J3; value Conn_01x04 -> Motor
- SW1: footprint Button_Switch_SMD:SW_Push_1TS009xxxx-xxxx-xxxx_6x6x5mm -> Button_Switch_SMD:SW_SPST_CK_RS282G05A3
Connections:
- net CRISTAL 1: now also C2.1
- net CRISTAL 2: now also C3.1; no longer C2.1
- net GND: now also C3.2
- net GND_MOT: now also C1.2; no longer D4.2 (A)
- net VCC_MOT: now also C1.1; no longer D2.1 (K)
- net RESET: now reaches R1.2, U1.1 (~{RESET}/PC6)
- net MotA2: now reaches A1.3 (A2), J2.1 (Pin_1)
- net MotA2: now also M1.2 (-)
- net MotA1: now reaches A1.4 (A1), J2.2 (Pin_2)
- net MotA1: now also M1.1
- net MotB1: now reaches A1.5 (B1), J2.3 (Pin_3)
- net MotB1: now also M1.3
- net MotB2: now reaches A1.6 (B2), J2.4 (Pin_4)
- net MotB2: now also M1.4
Other:
- note added: "Boton"
- note added: "Driver motor Paso A Paso"
- note added: "Microcontrolador ATMega328p"
- note added: "Motor Nema 17"
- note added: "Puente de diodos. Entrada AC -> Salida DC"
- note added: "Step Down 24 Lm2596 VC -> 5 VC"
- note removed: "Poder"
- company: (none) -> jm
- title: (none) -> arte.facto - Motorcin Bien Bemperado
- moved on the sheet: A1, D1, D2, D3, D4, H1, H2, H3, H4, J1, J2, R1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
